Commit message: 控制代码分层重构：仿真器无关算法核心 + ROS 适配层，实现 M1/M2 通道
- suspension_core.py：零 ROS 依赖控制核心，三个暴露面——参数面
  SuspensionConfig / 观测面 SuspensionInputs（含轮地接触）/ 动作面
  roll_ref+pitch_ref+height_cmd（Isaac Lab / RL 直接对接）
- active_suspension.py 改为薄适配层：参数自动声明、contact/{leg}
  与 ~/body_cmd 订阅、debug 扩展为 35 字段（前 22 字段布局不变）
- M2 车身高度通道（±0.06m 并入几何映射）、M1 接触保持状态机
  （悬空消抖→下探→撤回，受 target_limit 总限幅）——均默认关/零，
  默认参数下与 v3 逐步等价，待调参验收后启用
- 底盘外观改为模块化底盘视觉语言（载荷安装板+支撑柱+前保险杠，
  去整车造型），collision/惯量/关节零变更
- 冒烟验证：保持期零力矩、|tau| 严格 ≤ 120×0.45=54、适配层可导入

Co-Authored-By: Claude Fable 5 <noreply@anthropic.com>

File: src/tarantula_description/urdf/tarantula_chassis.xacro (robot description, xacro)
@@ -36,4 +36,7 @@
   <xacro:property name="pivot_y"      value="0.26"/>
   <xacro:property name="pivot_z"      value="-0.08"/>
+  <!-- 载荷安装板（模块化底盘的视觉/接口特征：平整安装面，非整车造型） -->
+  <xacro:property name="deck_standoff" value="0.03"/>   <!-- 支撑柱高 -->
+  <xacro:property name="deck_thick"    value="0.012"/>  <!-- 安装板厚 -->
   <xacro:property name="PI" value="3.14159265"/>
   <!-- ============ 惯量宏 ============ -->
@@ -45,4 +48,12 @@
     <inertia ixx="${m/12*(3*r*r+h*h)}" iyy="${m/12*(3*r*r+h*h)}" izz="${m/2*r*r}"
              ixy="0" ixz="0" iyz="0"/>
+  </xacro:macro>
+  <!-- 安装板支撑柱（视觉件） -->
+  <xacro:macro name="deck_post" params="x y">
+    <visual>
+      <origin xyz="${x} ${y} ${body_height/2 + deck_standoff/2}"/>
+      <geometry><cylinder radius="0.012" length="${deck_standoff}"/></geometry>
+      <xacro:mat_tire/>
+    </visual>
   </xacro:macro>
   <!-- 内联材质宏：RViz2 对命名材质引用渲染不可靠，必须逐 visual 内联颜色 -->
@@ -126,5 +137,7 @@
   <!-- ============ 底盘模块宏 ============ -->
   <xacro:macro name="tarantula_chassis" params="prefix:=''">
-    <!-- 车身：主舱 + 上层甲板 + 两侧悬挂安装梁 + 头部斜面 -->
+    <!-- 车身：主舱 + 载荷安装板（支撑柱架高的平整安装面）+ 两侧悬挂安装梁
+         + 前保险杠（方向标识）。视觉语言对标 Husky/Scout 类模块化底盘：
+         无整车造型，顶面就是给上装用的接口。只改 visual 不碰 collision。 -->
     <link name="${prefix}base_link">
       <visual>  <!-- 主舱 -->
@@ -132,12 +145,16 @@
         <xacro:mat_body/>
       </visual>
-      <visual>  <!-- 上层甲板 -->
-        <origin xyz="-0.05 0 ${body_height/2 + 0.03}"/>
-        <geometry><box size="0.45 0.28 0.06"/></geometry>
-        <xacro:mat_body/>
-      </visual>
-      <visual>  <!-- 头部斜面 -->
-        <origin xyz="${body_length/2 + 0.05} 0 0.01" rpy="0 0.35 0"/>
-        <geometry><box size="0.14 0.30 0.06"/></geometry>
+      <visual>  <!-- 载荷安装板 -->
+        <origin xyz="0 0 ${body_height/2 + deck_standoff + deck_thick/2}"/>
+        <geometry><box size="0.55 0.30 ${deck_thick}"/></geometry>
+        <xacro:mat_hub/>
+      </visual>
+      <xacro:deck_post x="0.24"  y="0.12"/>
+      <xacro:deck_post x="0.24"  y="-0.12"/>
+      <xacro:deck_post x="-0.24" y="0.12"/>
+      <xacro:deck_post x="-0.24" y="-0.12"/>
+      <visual>  <!-- 前保险杠 -->
+        <origin xyz="${body_length/2 + 0.015} 0 0"/>
+        <geometry><box size="0.03 ${body_width} 0.06"/></geometry>
         <xacro:mat_accent/>
       </visual>
@@ -172,5 +189,5 @@
       <origin xyz="0 0 ${body_height/2}"/>
     </joint>
-    <!-- 载荷安装位：外部载荷（LiDAR/相机/上装）统一挂这里，
+    <!-- 载荷安装位：安装板顶面中心，外部载荷（LiDAR/相机/上装）统一挂这里，
          底盘模块本身不预设任何载荷 -->
     <link name="${prefix}payload_mount"/>
@@ -178,5 +195,5 @@
       <parent link="${prefix}base_link"/>
       <child link="${prefix}payload_mount"/>
-      <origin xyz="0 0 ${body_height/2}"/>
+      <origin xyz="0 0 ${body_height/2 + deck_standoff + deck_thick}"/>
     </joint>
     <!-- 六条腿 -->

File: src/tarantula_description/urdf/tarantula_core.urdf.xacro (robot description, xacro)
@@ -36,5 +36,6 @@
       <parent link="payload_mount"/>
       <child link="lidar_link"/>
-      <origin xyz="0.22 0 0.12"/>
+      <!-- 安装板顶面(0.092) + 0.078 = 0.17，与历史 LiDAR 世界位姿严格一致 -->
+      <origin xyz="0.22 0 0.078"/>
     </joint>
   </xacro:if>
