Commit message: feat: add Isaac Lab RL v5 suspension policy

File: src/tarantula_description/urdf/tarantula.urdf.xacro (robot description, xacro)
@@ -1,8 +1,8 @@
 <?xml version="1.0"?>
 <!-- ============================================================
-     Gazebo Classic 适配层：include 本体（tarantula_core）后叠加
-     仿真器专属内容——物理弹簧标签、轮胎接触参数、传感器插件、
-     ros2_control。本体改动一律改 tarantula_core.urdf.xacro，
-     此文件只关心 Gazebo 的事。
+     Gazebo Ignition (gz-sim) 适配层：include 本体（tarantula_core）后叠加
+     仿真器专属内容——物理弹簧标签、轮胎接触参数、传感器、
+     ros2_control（经 gz_ros2_control）。本体改动一律改
+     tarantula_core.urdf.xacro，此文件只关心 Gazebo 的事。
      ============================================================ -->
 <robot xmlns:xacro="http://www.ros.org/wiki/xacro" name="tarantula">
@@ -11,11 +11,23 @@
   <xacro:macro name="leg_gazebo" params="prefix">
     <!-- 物理弹簧（被动悬挂硬件）：控制器未上线时车也能站立。
-         k 取自 core 的 susp_spring_k，与前馈刚度 ff_stiffness 严格一致 -->
+         k 取自 core 的 susp_spring_k，与前馈刚度 ff_stiffness 严格一致。
+         sdformat 将其转换为 SDF <axis><dynamics><spring_stiffness>/
+         <spring_reference>，dartsim 支持隐式弹簧阻尼。 -->
     <gazebo reference="susp_${prefix}_joint">
       <springStiffness>${susp_spring_k}</springStiffness>
       <springReference>0.0</springReference>
       <implicitSpringDamper>true</implicitSpringDamper>
+      <!-- 力/力矩传感器（存在性验证）：child(摆臂)对parent(车身)的反作用力，
+           用车身坐标表达——force.z 即该腿对车身的支撑力，>0 大致表示着地 -->
+      <sensor name="ft_${prefix}" type="force_torque">
+        <update_rate>50</update_rate>
+        <topic>ft/${prefix}</topic>
+        <force_torque>
+          <frame>parent</frame>
+          <measure_direction>child_to_parent</measure_direction>
+        </force_torque>
+      </sensor>
     </gazebo>
-    <!-- 轮胎接触参数 + 足端压力（接触）传感器 -->
+    <!-- 轮胎接触参数 -->
     <gazebo reference="wheel_${prefix}_link">
       <mu1>1.2</mu1>
@@ -23,20 +35,28 @@
       <kp>1000000.0</kp>
       <kd>100.0</kd>
-      <material>Gazebo/FlatBlack</material>
+    </gazebo>
+    <!-- 轮轴力/力矩传感器（验证用）：child(轮)对parent(摆臂)的反作用力，摆臂坐标表达。
+         轮子无弹簧、惯量远小于摆臂，理论上比髋关节 ft_${prefix} 更接近纯地面接触力，
+         用于对比噪声特征，暂不接入控制逻辑。 -->
+    <gazebo reference="wheel_${prefix}_joint">
+      <sensor name="ft_wheel_${prefix}" type="force_torque">
+        <update_rate>50</update_rate>
+        <topic>ft_wheel/${prefix}</topic>
+        <force_torque>
+          <frame>parent</frame>
+          <measure_direction>child_to_parent</measure_direction>
+        </force_torque>
+      </sensor>
+    </gazebo>
+    <!-- 几何接触传感器（地面真值）：wheel_${prefix}_link 的碰撞体是否与任意几何体接触，
+         与力/力矩信号在数值上无关——用于核查 force.z>阈值 是否真的对应"轮子着地"。 -->
+    <gazebo reference="wheel_${prefix}_link">
       <sensor name="contact_${prefix}" type="contact">
         <update_rate>50</update_rate>
+        <topic>contact/${prefix}</topic>
         <contact>
           <collision>wheel_${prefix}_link_collision</collision>
         </contact>
-        <plugin name="bumper_${prefix}" filename="libgazebo_ros_bumper.so">
-          <ros>
-            <remapping>bumper_states:=contact/${prefix}</remapping>
-          </ros>
-          <frame_name>wheel_${prefix}_link</frame_name>
-        </plugin>
       </sensor>
-    </gazebo>
-    <gazebo reference="arm_${prefix}_link">
-      <material>Gazebo/Orange</material>
     </gazebo>
   </xacro:macro>
@@ -48,7 +68,7 @@
   <xacro:leg_gazebo prefix="rr"/>
   <!-- ============ ros2_control ============ -->
-  <ros2_control name="GazeboSystem" type="system">
+  <ros2_control name="GazeboSimSystem" type="system">
     <hardware>
-      <plugin>gazebo_ros2_control/GazeboSystem</plugin>
+      <plugin>gz_ros2_control/GazeboSimSystem</plugin>
     </hardware>
     <xacro:macro name="susp_iface" params="prefix">
@@ -82,5 +102,5 @@
   <!-- ============ Gazebo 插件 ============ -->
   <gazebo>
-    <plugin filename="libgazebo_ros2_control.so" name="gazebo_ros2_control">
+    <plugin filename="gz_ros2_control-system" name="gz_ros2_control::GazeboSimROS2ControlPlugin">
       <parameters>$(find tarantula_bringup)/config/controllers.yaml</parameters>
     </plugin>
@@ -90,16 +110,12 @@
       <always_on>true</always_on>
       <update_rate>100</update_rate>
-      <plugin name="imu_plugin" filename="libgazebo_ros_imu_sensor.so">
-        <ros>
-          <remapping>~/out:=imu/data</remapping>
-        </ros>
-        <frame_name>imu_link</frame_name>
-      </plugin>
+      <topic>imu</topic>
     </sensor>
   </gazebo>
   <gazebo reference="lidar_link">
-    <sensor name="lidar_sensor" type="ray">
+    <sensor name="lidar_sensor" type="gpu_lidar">
       <always_on>true</always_on>
       <update_rate>10</update_rate>
+      <topic>scan</topic>
       <ray>
         <scan>
@@ -116,15 +132,5 @@
         </range>
       </ray>
-      <plugin name="lidar_plugin" filename="libgazebo_ros_ray_sensor.so">
-        <ros>
-          <remapping>~/out:=scan</remapping>
-        </ros>
-        <output_type>sensor_msgs/LaserScan</output_type>
-        <frame_name>lidar_link</frame_name>
-      </plugin>
     </sensor>
   </gazebo>
-  <gazebo reference="base_link">
-    <material>Gazebo/DarkGrey</material>
-  </gazebo>
 </robot>

Commit message: Align terrain and control baselines

File: src/tarantula_description/urdf/tarantula.urdf.xacro (robot description, xacro)
@@ -2,5 +2,5 @@
 <!-- ============================================================
      Gazebo Ignition (gz-sim) 适配层：include 本体（tarantula_core）后叠加
-     仿真器专属内容——物理弹簧标签、轮胎接触参数、传感器、
+     仿真器专属内容——轮胎接触参数、力/力矩传感器、
      ros2_control（经 gz_ros2_control）。本体改动一律改
      tarantula_core.urdf.xacro，此文件只关心 Gazebo 的事。
@@ -10,14 +10,7 @@
   <!-- ============ 每腿 Gazebo 标签 ============ -->
   <xacro:macro name="leg_gazebo" params="prefix">
-    <!-- 物理弹簧（被动悬挂硬件）：控制器未上线时车也能站立。
-         k 取自 core 的 susp_spring_k，与前馈刚度 ff_stiffness 严格一致。
-         sdformat 将其转换为 SDF <axis><dynamics><spring_stiffness>/
-         <spring_reference>，dartsim 支持隐式弹簧阻尼。 -->
+    <!-- 髋关节力/力矩传感器：child(摆臂)对parent(车身)的反作用力。
+         只做诊断/系统辨识，不作为部署策略的必需接触真值。 -->
     <gazebo reference="susp_${prefix}_joint">
-      <springStiffness>${susp_spring_k}</springStiffness>
-      <springReference>0.0</springReference>
-      <implicitSpringDamper>true</implicitSpringDamper>
-      <!-- 力/力矩传感器（存在性验证）：child(摆臂)对parent(车身)的反作用力，
-           用车身坐标表达——force.z 即该腿对车身的支撑力，>0 大致表示着地 -->
       <sensor name="ft_${prefix}" type="force_torque">
         <update_rate>50</update_rate>
@@ -31,12 +24,11 @@
     <!-- 轮胎接触参数 -->
     <gazebo reference="wheel_${prefix}_link">
-      <mu1>1.2</mu1>
-      <mu2>0.8</mu2>
+      <mu1>1.35</mu1>
+      <mu2>1.05</mu2>
       <kp>1000000.0</kp>
-      <kd>100.0</kd>
+      <kd>140.0</kd>
     </gazebo>
-    <!-- 轮轴力/力矩传感器（验证用）：child(轮)对parent(摆臂)的反作用力，摆臂坐标表达。
-         轮子无弹簧、惯量远小于摆臂，理论上比髋关节 ft_${prefix} 更接近纯地面接触力，
-         用于对比噪声特征，暂不接入控制逻辑。 -->
+    <!-- 轮轴力/力矩传感器：部署可实现的轮载观测来源（轮毂/轮轴 F/T）。
+         RL 不使用几何 contact boolean；轮载由 ||F|| 或法向力连续估计。 -->
     <gazebo reference="wheel_${prefix}_joint">
       <sensor name="ft_wheel_${prefix}" type="force_torque">
@@ -47,15 +39,4 @@
           <measure_direction>child_to_parent</measure_direction>
         </force_torque>
-      </sensor>
-    </gazebo>
-    <!-- 几何接触传感器（地面真值）：wheel_${prefix}_link 的碰撞体是否与任意几何体接触，
-         与力/力矩信号在数值上无关——用于核查 force.z>阈值 是否真的对应"轮子着地"。 -->
-    <gazebo reference="wheel_${prefix}_link">
-      <sensor name="contact_${prefix}" type="contact">
-        <update_rate>50</update_rate>
-        <topic>contact/${prefix}</topic>
-        <contact>
-          <collision>wheel_${prefix}_link_collision</collision>
-        </contact>
       </sensor>
     </gazebo>

File: src/tarantula_description/urdf/tarantula_chassis.xacro (robot description, xacro)
@@ -21,14 +21,26 @@
   <xacro:property name="body_height"  value="0.10"/>
   <xacro:property name="body_mass"    value="18.0"/>
+  <!-- COM 显式参数化，便于 Isaac/Gazebo 域随机化和载荷敏感性实验对齐。 -->
+  <xacro:property name="body_com_x"   value="0.0"/>
+  <xacro:property name="body_com_y"   value="0.0"/>
+  <xacro:property name="body_com_z"   value="-0.025"/>
+  <!-- 物理碰撞略小于视觉外壳，避免托底/擦边时用装饰外形参与接触。 -->
+  <xacro:property name="belly_length" value="0.70"/>
+  <xacro:property name="belly_width"  value="0.30"/>
+  <xacro:property name="belly_height" value="0.08"/>
+  <xacro:property name="belly_z"      value="0.015"/>
   <xacro:property name="arm_length"   value="0.22"/>   <!-- 悬挂摆臂长度 -->
   <xacro:property name="arm_mass"     value="0.8"/>
   <xacro:property name="arm_angle"    value="0.698"/>  <!-- 摆臂下倾 40 度 -->
-  <xacro:property name="wheel_radius" value="0.12"/>
-  <xacro:property name="wheel_width"  value="0.07"/>
-  <xacro:property name="wheel_mass"   value="1.5"/>
-  <!-- 悬挂物理弹簧/阻尼（被动层硬件参数，主动控制的前馈刚度必须与 k 一致） -->
-  <xacro:property name="susp_spring_k"  value="120.0"/> <!-- Nm/rad -->
-  <xacro:property name="susp_damping"   value="8.0"/>   <!-- Nms/rad -->
-  <xacro:property name="susp_friction"  value="0.1"/>
+  <xacro:property name="wheel_radius" value="0.13"/>
+  <xacro:property name="wheel_width"  value="0.075"/>
+  <xacro:property name="wheel_mass"   value="1.7"/>
+  <!-- 轮胎视觉保持圆柱。碰撞体默认用 sphere；cylinder 仅保留为已知失败对照。 -->
+  <xacro:property name="wheel_collision_radius" value="${wheel_radius}"/>
+  <!-- 悬挂执行器等效 PD 参数。论文式 RL 部署不依赖 Gazebo-only joint spring，
+       Gazebo/Isaac 都应通过受限执行器把目标角转换为力矩。 -->
+  <xacro:property name="susp_actuator_kp" value="130.0"/> <!-- Nm/rad -->
+  <xacro:property name="susp_damping"   value="11.0"/>  <!-- Nms/rad -->
+  <xacro:property name="susp_friction"  value="0.08"/>
   <!-- 蜘蛛站姿：前腿朝前(dir=+1)、中后腿朝后(dir=-1)，六轮均布 x=+0.51/0/-0.51 -->
   <xacro:property name="pivot_x"      value="0.34"/>
@@ -66,5 +78,5 @@
        悬挂关节绕 y 轴，轮关节绕 y 轴连续转动。
        注意：dir 决定关节角与轮子升降的方向关系，控制节点 DIR 表必须一致。 -->
-  <xacro:macro name="leg" params="prefix id x side dir">
+  <xacro:macro name="leg" params="prefix id x side dir wheel_collision">
     <joint name="${prefix}susp_${id}_joint" type="revolute">
       <parent link="${prefix}base_link"/>
@@ -72,5 +84,5 @@
       <origin xyz="${x} ${side*pivot_y} ${pivot_z}" rpy="0 0 0"/>
       <axis xyz="0 1 0"/>
-      <limit lower="-0.6" upper="0.6" effort="60" velocity="6"/>
+      <limit lower="-0.6" upper="0.6" effort="75" velocity="6"/>
       <!-- 阻尼放物理侧（无控制延迟），软件 PD 的 kd 对延迟敏感不可依赖 -->
       <dynamics damping="${susp_damping}" friction="${susp_friction}"/>
@@ -110,6 +122,6 @@
       <origin xyz="${dir*arm_length*cos(arm_angle)} ${side*0.065} ${-arm_length*sin(arm_angle)}"/>
       <axis xyz="0 1 0"/>
-      <limit effort="30" velocity="30"/>
-      <dynamics damping="0.1"/>
+      <limit effort="38" velocity="30"/>
+      <dynamics damping="0.08"/>
     </joint>
     <link name="${prefix}wheel_${id}_link">
@@ -124,8 +136,15 @@
         <xacro:mat_hub/>
       </visual>
-      <collision>
-        <origin rpy="${PI/2} 0 0"/>
-        <geometry><cylinder radius="${wheel_radius}" length="${wheel_width}"/></geometry>
-      </collision>
+      <xacro:if value="${wheel_collision == 'sphere'}">
+        <collision name="wheel_${id}_contact_collision">
+          <geometry><sphere radius="${wheel_collision_radius}"/></geometry>
+        </collision>
+      </xacro:if>
+      <xacro:if value="${wheel_collision == 'cylinder'}">
+        <collision name="wheel_${id}_contact_collision">
+          <origin rpy="${PI/2} 0 0"/>
+          <geometry><cylinder radius="${wheel_radius}" length="${wheel_width}"/></geometry>
+        </collision>
+      </xacro:if>
       <inertial>
         <origin rpy="${PI/2} 0 0"/>
@@ -136,5 +155,5 @@
   </xacro:macro>
   <!-- ============ 底盘模块宏 ============ -->
-  <xacro:macro name="tarantula_chassis" params="prefix:=''">
+  <xacro:macro name="tarantula_chassis" params="prefix:='' wheel_collision:='sphere'">
     <!-- 车身：主舱 + 载荷安装板（支撑柱架高的平整安装面）+ 两侧悬挂安装梁
          + 前保险杠（方向标识）。视觉语言对标 Husky/Scout 类模块化底盘：
@@ -169,8 +188,10 @@
         <xacro:mat_accent/>
       </visual>
-      <collision>
-        <geometry><box size="${body_length} ${body_width} ${body_height}"/></geometry>
+      <collision name="base_belly_collision">
+        <origin xyz="0 0 ${belly_z}"/>
+        <geometry><box size="${belly_length} ${belly_width} ${belly_height}"/></geometry>
       </collision>
       <inertial>
+        <origin xyz="${body_com_x} ${body_com_y} ${body_com_z}"/>
         <mass value="${body_mass}"/>
         <xacro:box_inertia m="${body_mass}" x="${body_length}" y="${body_width}" z="${body_height}"/>
@@ -198,10 +219,10 @@
     </joint>
     <!-- 六条腿 -->
-    <xacro:leg prefix="${prefix}" id="fl" x="${pivot_x}"  side="1"  dir="1"/>
-    <xacro:leg prefix="${prefix}" id="fr" x="${pivot_x}"  side="-1" dir="1"/>
-    <xacro:leg prefix="${prefix}" id="ml" x="${pivot_mx}" side="1"  dir="-1"/>
-    <xacro:leg prefix="${prefix}" id="mr" x="${pivot_mx}" side="-1" dir="-1"/>
-    <xacro:leg prefix="${prefix}" id="rl" x="${-pivot_x}" side="1"  dir="-1"/>
-    <xacro:leg prefix="${prefix}" id="rr" x="${-pivot_x}" side="-1" dir="-1"/>
+    <xacro:leg prefix="${prefix}" id="fl" x="${pivot_x}"  side="1"  dir="1"  wheel_collision="${wheel_collision}"/>
+    <xacro:leg prefix="${prefix}" id="fr" x="${pivot_x}"  side="-1" dir="1"  wheel_collision="${wheel_collision}"/>
+    <xacro:leg prefix="${prefix}" id="ml" x="${pivot_mx}" side="1"  dir="-1" wheel_collision="${wheel_collision}"/>
+    <xacro:leg prefix="${prefix}" id="mr" x="${pivot_mx}" side="-1" dir="-1" wheel_collision="${wheel_collision}"/>
+    <xacro:leg prefix="${prefix}" id="rl" x="${-pivot_x}" side="1"  dir="-1" wheel_collision="${wheel_collision}"/>
+    <xacro:leg prefix="${prefix}" id="rr" x="${-pivot_x}" side="-1" dir="-1" wheel_collision="${wheel_collision}"/>
   </xacro:macro>
 </robot>

File: src/tarantula_description/urdf/tarantula_core.urdf.xacro (robot description, xacro)
@@ -8,11 +8,13 @@
        xacro tarantula_core.urdf.xacro > tarantula.urdf          # 带 LiDAR
        xacro tarantula_core.urdf.xacro lidar:=false > bare.urdf  # 裸底盘
-     悬挂物理弹簧 k=120 Nm/rad、阻尼 c=8 在 Isaac 中映射为关节
-     drive 的 stiffness/damping（隐式 PD，与 Gazebo
-     implicitSpringDamper 同角色），见 docs §7。
+       xacro tarantula_core.urdf.xacro wheel_collision:=cylinder # 圆柱 collision A/B
+     悬挂执行器等效参数 kp=120 Nm/rad、kd=8 Nms/rad 在 Isaac 中映射为
+     关节 drive 的 stiffness/damping；Gazebo 部署侧由策略节点显式计算
+     受限 PD 力矩，不再依赖 Gazebo-only joint spring。
      ============================================================ -->
 <robot xmlns:xacro="http://www.ros.org/wiki/xacro" name="tarantula">
   <xacro:include filename="$(find tarantula_description)/urdf/tarantula_chassis.xacro"/>
-  <xacro:tarantula_chassis prefix=""/>
+  <xacro:arg name="wheel_collision" default="sphere"/>
+  <xacro:tarantula_chassis prefix="" wheel_collision="$(arg wheel_collision)"/>
   <!-- ============ LiDAR 载荷（可选，挂 payload_mount） ============ -->
   <xacro:arg name="lidar" default="true"/>
@@ -36,5 +38,5 @@
       <parent link="payload_mount"/>
       <child link="lidar_link"/>
-      <!-- 安装板顶面(0.092) + 0.078 = 0.17，与历史 LiDAR 世界位姿严格一致 -->
+      <!-- 安装板顶面(0.092) + 0.078 = 0.17 -->
       <origin xyz="0.22 0 0.078"/>
     </joint>
