Commit message: Set stage B RL baseline and benchmark gates

File: src/tarantula_description/urdf/tarantula_chassis_v2.xacro (robot description, xacro)
@@ -94,5 +94,5 @@
     </link>
   </xacro:macro>
-  <xacro:macro name="tarantula_chassis_v2" params="prefix:='' wheel_collision:='cylinder'">
+  <xacro:macro name="tarantula_chassis_v2" params="prefix:='' wheel_collision:='sphere'">
     <link name="${prefix}base_link">
       <visual><geometry><box size="${body_length} ${body_width} ${body_height}"/></geometry><xacro:mat_body/></visual>

File: src/tarantula_description/urdf/tarantula_core_v2.urdf.xacro (robot description, xacro)
@@ -2,5 +2,5 @@
 <robot xmlns:xacro="http://www.ros.org/wiki/xacro" name="tarantula">
   <xacro:include filename="$(find tarantula_description)/urdf/tarantula_chassis_v2.xacro"/>
-  <xacro:arg name="wheel_collision" default="cylinder"/>
+  <xacro:arg name="wheel_collision" default="sphere"/>
   <xacro:tarantula_chassis_v2 prefix="" wheel_collision="$(arg wheel_collision)"/>
   <xacro:arg name="lidar" default="true"/>
